File: psu.sch (KiCad schematic (older format))
At the start: 0 parts

Commit message: ch1 and ch2 are complete
Parts:
- added C301, C302, C507, C508, C509, C510: 100n, Capacitor_SMD:C_1206_3216Metric_Pad1.42x1.75mm_HandSolder, symbol Device:C_Small
- added C503, C504: 47uF, Capacitor_THT:CP_Radial_D6.3mm_P2.50mm, symbol Device:CP_Small
- added C505, C506: 470uF, Capacitor_THT:CP_Radial_D10.0mm_P5.00mm, symbol Device:CP_Small
- added D301, D302, D303, D304: M7, Diode_SMD:D_SMA_Handsoldering, symbol Device:D
- added J501: POWER, TerminalBlock_Phoenix:TerminalBlock_Phoenix_PT-1,5-3-3.5-H_1x03_P3.50mm_Horizontal, symbol Connector:Screw_Terminal_01x03
- added R501, R504: 120R, Resistor_SMD:R_0805_2012Metric_Pad1.15x1.40mm_HandSolder, symbol Device:R_Small
- added R502, R503: 1K4, Resistor_SMD:R_0805_2012Metric_Pad1.15x1.40mm_HandSolder, symbol Device:R_Small
- added U301: LM317_TO-252, Package_TO_SOT_SMD:TO-252-2, symbol Regulator_Linear:LM317_TO-252
- added U302: LM337_TO252, Package_TO_SOT_SMD:TO-252-2, symbol Regulator_Linear:LM337_TO252
Connections:
- new net +15V: C505.1, C507.1, C509.1, D301.2 (A), D303.1 (K), R501.1, U301.2 (VO)
- new net -15V: C506.2, C508.2, C510.2, D302.1 (K), D304.2 (A), R504.2, U302.3 (VO)
- new net 317ADJ: C503.1, D303.2 (A), R501.2, R502.1, U301.1 (ADJ)
- new net 337ADJ: C504.2, D304.1 (K), R503.2, R504.1, U302.1 (ADJ)
- new net GND: C301.2, C302.1, C503.2, C504.1, C505.2, C506.1, C507.2, C508.1, C509.2, C510.1, J501.2 (Pin_2), R502.2, R503.1
- new net V+: C301.1, D301.1 (K), J501.1 (Pin_1), U301.3 (VI)
- new net V-: C302.2, D302.2 (A), J501.3 (Pin_3), U302.2 (VI)
Other:
- note added: "pg 3xx"

Commit message: assigned footprints
Parts:
- D301, D302, D303, D304: footprint Diode_SMD:D_SMA_Handsoldering -> Diode_SMD:D_SMA
Changed lines of the file:
@@
 F 0 "D301" H 4000 2817 50  0000 C CNN
 F 1 "M7" H 4000 2726 50  0000 C CNN
-F 2 "Diode_SMD:D_SMA_Handsoldering" H 4000 2600 50  0001 C CNN
+F 2 "Diode_SMD:D_SMA" H 4000 2600 50  0001 C CNN
 F 3 "~" H 4000 2600 50  0001 C CNN
 	1    4000 2600
@@
 F 0 "D303" V 4954 3330 50  0000 L CNN
 F 1 "M7" V 5045 3330 50  0000 L CNN
-F 2 "Diode_SMD:D_SMA_Handsoldering" H 5000 3250 50  0001 C CNN
+F 2 "Diode_SMD:D_SMA" H 5000 3250 50  0001 C CNN
 F 3 "~" H 5000 3250 50  0001 C CNN
 	1    5000 3250
@@
 F 0 "D304" V 4954 4830 50  0000 L CNN
 F 1 "M7" V 5045 4830 50  0000 L CNN
-F 2 "Diode_SMD:D_SMA_Handsoldering" H 5000 4750 50  0001 C CNN
+F 2 "Diode_SMD:D_SMA" H 5000 4750 50  0001 C CNN
 F 3 "~" H 5000 4750 50  0001 C CNN
 	1    5000 4750
@@
 F 0 "D302" H 4000 5383 50  0000 C CNN
 F 1 "M7" H 4000 5474 50  0000 C CNN
-F 2 "Diode_SMD:D_SMA_Handsoldering" H 4000 5600 50  0001 C CNN
+F 2 "Diode_SMD:D_SMA" H 4000 5600 50  0001 C CNN
 F 3 "~" H 4000 5600 50  0001 C CNN
 	1    4000 5600
@@
 $EndComp
 $Comp
-L power:GND #PWR012
+L power:GND #PWR0103
 U 1 1 648F1D4C
 P 7000 4100
-F 0 "#PWR012" H 7000 3850 50  0001 C CNN
+F 0 "#PWR0103" H 7000 3850 50  0001 C CNN
 F 1 "GND" H 7005 3927 50  0000 C CNN
 F 2 "" H 7000 4100 50  0001 C CNN

Commit message: pcb started
Parts:
- added C511, C512, C513, C514: 100n, Capacitor_SMD:C_1206_3216Metric_Pad1.42x1.75mm_HandSolder, symbol Device:C_Small
Connections:
- net +15V: now also C511.1, C513.1
- net -15V: now also C512.2, C514.2
- net GND: now also C511.2, C512.1, C513.2, C514.1
Changed lines of the file:
@@
 L power:GND #PWR0103
 U 1 1 648F1D4C
-P 7000 4100
-F 0 "#PWR0103" H 7000 3850 50  0001 C CNN
-F 1 "GND" H 7005 3927 50  0000 C CNN
-F 2 "" H 7000 4100 50  0001 C CNN
-F 3 "" H 7000 4100 50  0001 C CNN
-	1    7000 4100
+P 7800 4000
+F 0 "#PWR0103" H 7800 3750 50  0001 C CNN
+F 1 "GND" H 7805 3827 50  0000 C CNN
+F 2 "" H 7800 4000 50  0001 C CNN
+F 3 "" H 7800 4000 50  0001 C CNN
+	1    7800 4000
 	1    0    0    -1
 $EndComp
@@
 L power:+15V #PWR0105
 U 1 1 646FA71D
-P 6500 2850
-F 0 "#PWR0105" H 6500 2700 50  0001 C CNN
-F 1 "+15V" H 6515 3023 50  0000 C CNN
-F 2 "" H 6500 2850 50  0001 C CNN
-F 3 "" H 6500 2850 50  0001 C CNN
-	1    6500 2850
+P 7500 2900
+F 0 "#PWR0105" H 7500 2750 50  0001 C CNN
+F 1 "+15V" H 7515 3073 50  0000 C CNN
+F 2 "" H 7500 2900 50  0001 C CNN
+F 3 "" H 7500 2900 50  0001 C CNN
+	1    7500 2900
 	1    0    0    -1
 $EndComp
@@
 	6000 3000 6500 3000
 Wire Wire Line
-	7000 4100 7000 4000
-Wire Wire Line
-	7000 4000 6500 4000
-Wire Wire Line
 	6000 3600 6000 4000
 Connection ~ 6000 4000
@@
 L power:-15V #PWR0106
 U 1 1 6470844E
-P 6500 5150
-F 0 "#PWR0106" H 6500 5250 50  0001 C CNN
-F 1 "-15V" H 6515 5323 50  0000 C CNN
-F 2 "" H 6500 5150 50  0001 C CNN
-F 3 "" H 6500 5150 50  0001 C CNN
-	1    6500 5150
+P 7500 5100
+F 0 "#PWR0106" H 7500 5200 50  0001 C CNN
+F 1 "-15V" H 7515 5273 50  0000 C CNN
+F 2 "" H 7500 5100 50  0001 C CNN
+F 3 "" H 7500 5100 50  0001 C CNN
+	1    7500 5100
 	-1   0    0    1
 $EndComp
-Wire Wire Line
-	6500 5150 6500 5000
-Connection ~ 6500 5000
-Wire Wire Line
-	6500 2850 6500 3000
-Connection ~ 6500 3000
 Wire Wire Line
 	6000 4600 6000 5000
@@
 Wire Wire Line
 	6000 5000 5500 5000
+$Comp
+L Device:C_Small C512
+U 1 1 6476B82D
+P 7000 4500
+F 0 "C512" H 7092 4546 50  0000 L CNN
+F 1 "100n" H 7092 4455 50  0000 L CNN
+F 2 "Capacitor_SMD:C_1206_3216Metric_Pad1.42x1.75mm_HandSolder" H 7000 4500 50  0001 C CNN
+F 3 "~" H 7000 4500 50  0001 C CNN
+	1    7000 4500
+	1    0    0    -1
+$EndComp
+$Comp
+L Device:C_Small C514
+U 1 1 6476BE66
+P 7500 4500
+F 0 "C514" H 7592 4546 50  0000 L CNN
+F 1 "100n" H 7592 4455 50  0000 L CNN
+F 2 "Capacitor_SMD:C_1206_3216Metric_Pad1.42x1.75mm_HandSolder" H 7500 4500 50  0001 C CNN
+F 3 "~" H 7500 4500 50  0001 C CNN
+	1    7500 4500
+	1    0    0    -1
+$EndComp
+$Comp
+L Device:C_Small C511
+U 1 1 6476C2A5
+P 7000 3500
+F 0 "C511" H 7092 3546 50  0000 L CNN
+F 1 "100n" H 7092 3455 50  0000 L CNN
+F 2 "Capacitor_SMD:C_1206_3216Metric_Pad1.42x1.75mm_HandSolder" H 7000 3500 50  0001 C CNN
+F 3 "~" H 7000 3500 50  0001 C CNN
+	1    7000 3500
+	1    0    0    -1
+$EndComp
+$Comp
+L Device:C_Small C513
+U 1 1 6476C90C
+P 7500 3500
+F 0 "C513" H 7592 3546 50  0000 L CNN
+F 1 "100n" H 7592 3455 50  0000 L CNN
+F 2 "Capacitor_SMD:C_1206_3216Metric_Pad1.42x1.75mm_HandSolder" H 7500 3500 50  0001 C CNN
+F 3 "~" H 7500 3500 50  0001 C CNN
+	1    7500 3500
+	1    0    0    -1
+$EndComp
+Wire Wire Line
+	7500 3600 7500 4000
+Wire Wire Line
+	7500 4000 7000 4000
+Wire Wire Line
+	7500 4400 7500 4000
+Connection ~ 7500 4000
+Wire Wire Line
+	7500 4600 7500 5000
+Wire Wire Line
+	7500 5000 7000 5000
+Connection ~ 6500 5000
+Wire Wire Line
+	7000 4600 7000 5000
+Connection ~ 7000 5000
+Wire Wire Line
+	7000 5000 6500 5000
+Wire Wire Line
+	7000 4400 7000 4000
+Connection ~ 7000 4000
+Wire Wire Line
+	7000 4000 6500 4000
+Wire Wire Line
+	7000 3600 7000 4000
+Wire Wire Line
+	7500 3400 7500 3000
+Wire Wire Line
+	7500 3000 7000 3000
+Connection ~ 6500 3000
+Wire Wire Line
+	7000 3400 7000 3000
+Connection ~ 7000 3000
+Wire Wire Line
+	7000 3000 6500 3000
+Wire Wire Line
+	7500 5100 7500 5000
+Connection ~ 7500 5000
+Wire Wire Line
+	7500 2900 7500 3000
+Connection ~ 7500 3000
+Wire Wire Line
+	7800 4000 7500 4000
 $EndSCHEMATC

Commit message: pcb layout
Parts:
- renumbered C503 to C303, C504 to C304, C505 to C305, C506 to C306, C507 to C307, C508 to C308, C509 to C309, C510 to C310, C511 to C311, C512 to C312, C513 to C313, C514 to C314, R501 to R301, R502 to R302, R503 to R303, R504 to R304
Changed lines of the file:
@@
 $EndComp
 $Comp
-L Device:R_Small R501
+L Device:R_Small R301
 U 1 1 648E8C82
 P 4500 3250
-F 0 "R501" H 4559 3296 50  0000 L CNN
+F 0 "R301" H 4559 3296 50  0000 L CNN
 F 1 "120R" H 4559 3205 50  0000 L CNN
 F 2 "Resistor_SMD:R_0805_2012Metric_Pad1.15x1.40mm_HandSolder" H 4500 3250 50  0001 C CNN
@@
 $EndComp
 $Comp
-L Device:R_Small R502
+L Device:R_Small R302
 U 1 1 648E964A
 P 4500 3750
-F 0 "R502" H 4559 3796 50  0000 L CNN
+F 0 "R302" H 4559 3796 50  0000 L CNN
 F 1 "1K4" H 4559 3705 50  0000 L CNN
 F 2 "Resistor_SMD:R_0805_2012Metric_Pad1.15x1.40mm_HandSolder" H 4500 3750 50  0001 C CNN
@@
 $EndComp
 $Comp
-L Device:CP_Small C503
+L Device:CP_Small C303
 U 1 1 648E9C5F
 P 5000 3750
-F 0 "C503" H 5088 3796 50  0000 L CNN
+F 0 "C303" H 5088 3796 50  0000 L CNN
 F 1 "47uF" H 5088 3705 50  0000 L CNN
 F 2 "Capacitor_THT:CP_Radial_D6.3mm_P2.50mm" H 5000 3750 50  0001 C CNN
@@
 $EndComp
 $Comp
-L Device:CP_Small C505
+L Device:CP_Small C305
 U 1 1 648EA75B
 P 5500 3500
-F 0 "C505" H 5588 3546 50  0000 L CNN
+F 0 "C305" H 5588 3546 50  0000 L CNN
 F 1 "470uF" H 5588 3455 50  0000 L CNN
 F 2 "Capacitor_THT:CP_Radial_D10.0mm_P5.00mm" H 5500 3500 50  0001 C CNN
@@
 $EndComp
 $Comp
-L Device:R_Small R504
+L Device:R_Small R304
 U 1 1 648EB629
 P 4500 4750
-F 0 "R504" H 4559 4796 50  0000 L CNN
+F 0 "R304" H 4559 4796 50  0000 L CNN
 F 1 "120R" H 4559 4705 50  0000 L CNN
 F 2 "Resistor_SMD:R_0805_2012Metric_Pad1.15x1.40mm_HandSolder" H 4500 4750 50  0001 C CNN
@@
 $EndComp
 $Comp
-L Device:R_Small R503
+L Device:R_Small R303
 U 1 1 648EBE0F
 P 4500 4250
-F 0 "R503" H 4559 4296 50  0000 L CNN
+F 0 "R303" H 4559 4296 50  0000 L CNN
 F 1 "1K4" H 4559 4205 50  0000 L CNN
 F 2 "Resistor_SMD:R_0805_2012Metric_Pad1.15x1.40mm_HandSolder" H 4500 4250 50  0001 C CNN
@@
 $EndComp
 $Comp
-L Device:CP_Small C504
+L Device:CP_Small C304
 U 1 1 648EC340
 P 5000 4250
-F 0 "C504" H 5088 4296 50  0000 L CNN
+F 0 "C304" H 5088 4296 50  0000 L CNN
 F 1 "47uF" H 5088 4205 50  0000 L CNN
 F 2 "Capacitor_THT:CP_Radial_D6.3mm_P2.50mm" H 5000 4250 50  0001 C CNN
@@
 $EndComp
 $Comp
-L Device:CP_Small C506
+L Device:CP_Small C306
 U 1 1 648ED375
 P 5500 4500
-F 0 "C506" H 5588 4546 50  0000 L CNN
+F 0 "C306" H 5588 4546 50  0000 L CNN
 F 1 "470uF" H 5588 4455 50  0000 L CNN
 F 2 "Capacitor_THT:CP_Radial_D10.0mm_P5.00mm" H 5500 4500 50  0001 C CNN
@@
 pg 3xx
 $Comp
-L Device:C_Small C507
+L Device:C_Small C307
 U 1 1 646F5CB1
 P 6000 3500
-F 0 "C507" H 6092 3546 50  0000 L CNN
+F 0 "C307" H 6092 3546 50  0000 L CNN
 F 1 "100n" H 6092 3455 50  0000 L CNN
 F 2 "Capacitor_SMD:C_1206_3216Metric_Pad1.42x1.75mm_HandSolder" H 6000 3500 50  0001 C CNN
@@
 $EndComp
 $Comp
-L Device:C_Small C509
+L Device:C_Small C309
 U 1 1 646F666B
 P 6500 3500
-F 0 "C509" H 6592 3546 50  0000 L CNN
+F 0 "C309" H 6592 3546 50  0000 L CNN
 F 1 "100n" H 6592 3455 50  0000 L CNN
 F 2 "Capacitor_SMD:C_1206_3216Metric_Pad1.42x1.75mm_HandSolder" H 6500 3500 50  0001 C CNN
@@
 $EndComp
 $Comp
-L Device:C_Small C508
+L Device:C_Small C308
 U 1 1 646F6C31
 P 6000 4500
-F 0 "C508" H 6092 4546 50  0000 L CNN
+F 0 "C308" H 6092 4546 50  0000 L CNN
 F 1 "100n" H 6092 4455 50  0000 L CNN
 F 2 "Capacitor_SMD:C_1206_3216Metric_Pad1.42x1.75mm_HandSolder" H 6000 4500 50  0001 C CNN
@@
 $EndComp
 $Comp
-L Device:C_Small C510
+L Device:C_Small C310
 U 1 1 646F7253
 P 6500 4500
-F 0 "C510" H 6592 4546 50  0000 L CNN
+F 0 "C310" H 6592 4546 50  0000 L CNN
 F 1 "100n" H 6592 4455 50  0000 L CNN
 F 2 "Capacitor_SMD:C_1206_3216Metric_Pad1.42x1.75mm_HandSolder" H 6500 4500 50  0001 C CNN
@@
 	6000 5000 5500 5000
 $Comp
-L Device:C_Small C512
+L Device:C_Small C312
 U 1 1 6476B82D
 P 7000 4500
-F 0 "C512" H 7092 4546 50  0000 L CNN
+F 0 "C312" H 7092 4546 50  0000 L CNN
 F 1 "100n" H 7092 4455 50  0000 L CNN
 F 2 "Capacitor_SMD:C_1206_3216Metric_Pad1.42x1.75mm_HandSolder" H 7000 4500 50  0001 C CNN
@@
 $EndComp
 $Comp
-L Device:C_Small C514
+L Device:C_Small C314
 U 1 1 6476BE66
 P 7500 4500
-F 0 "C514" H 7592 4546 50  0000 L CNN
+F 0 "C314" H 7592 4546 50  0000 L CNN
 F 1 "100n" H 7592 4455 50  0000 L CNN
 F 2 "Capacitor_SMD:C_1206_3216Metric_Pad1.42x1.75mm_HandSolder" H 7500 4500 50  0001 C CNN
@@
 $EndComp
 $Comp
-L Device:C_Small C511
+L Device:C_Small C311
 U 1 1 6476C2A5
 P 7000 3500
-F 0 "C511" H 7092 3546 50  0000 L CNN
+F 0 "C311" H 7092 3546 50  0000 L CNN
 F 1 "100n" H 7092 3455 50  0000 L CNN
 F 2 "Capacitor_SMD:C_1206_3216Metric_Pad1.42x1.75mm_HandSolder" H 7000 3500 50  0001 C CNN
@@
 $EndComp
 $Comp
-L Device:C_Small C513
+L Device:C_Small C313
 U 1 1 6476C90C
 P 7500 3500
-F 0 "C513" H 7592 3546 50  0000 L CNN
+F 0 "C313" H 7592 3546 50  0000 L CNN
 F 1 "100n" H 7592 3455 50  0000 L CNN
 F 2 "Capacitor_SMD:C_1206_3216Metric_Pad1.42x1.75mm_HandSolder" H 7500 3500 50  0001 C CNN
