File: input_buffer_discrete.kicad_pcb (KiCad board)
At the start: 2 copper layers, 119 parts, among them J101 CH1, J102 CH1OUT, J2 CH2, J301 POWER, J4 CH2OUT, Q101 BC856BDW1, Q102 LS844, Q103 BC846BDW1, Q104 BC856, Q105 BCP53, Q106 BC846, Q107 BCP56, Q111 BC856BDW1, Q112 LS844, Q113 BC846BDW1, Q114 BC856, Q115 BCP53, Q116 BC846, Q117 BCP56, Q201 BC856BDW1, Q202 LS844, Q203 BC846BDW1, Q204 BC856, Q205 BCP53, Q206 BC846, Q207 BCP56, Q211 BC856BDW1, Q212 LS844, Q213 BC846BDW1, Q214 BC856, Q215 BCP53, Q216 BC846, Q217 BCP56, U301 LM317_TO-252, U302 LM337_TO252

Commit message: pcb started
Parts:
- removed C10, C9: 680p, Capacitor_SMD:C_0805_2012Metric_Pad1.15x1.40mm_HandSolder
- removed the C103 at (60.8, 123.8)
- removed the C105 at (81.5, 103.0)
- removed the R108 at (63.2, 123.8)
- removed the R116 at (53.2, 67.8)
- removed the R119 at (81.0, 108.2)
- removed R127, R53, R54: 100R, Resistor_SMD:R_0805_2012Metric_Pad1.15x1.40mm_HandSolder
- removed R39, R40: 470R, Resistor_SMD:R_0805_2012Metric_Pad1.15x1.40mm_HandSolder
- added C101: 10u, Capacitor_THT:C_Radial_D5.0mm_H7.0mm_P2.00mm, F.Cu at (63.0, 122.8)
- added C102: 10u, Capacitor_THT:C_Radial_D5.0mm_H7.0mm_P2.00mm, F.Cu at (87.0, 122.8)
- added C201: 10u, Capacitor_THT:C_Radial_D5.0mm_H7.0mm_P2.00mm, F.Cu at (104.8, 134.6)
- added C202: 10u, Capacitor_THT:C_Radial_D5.0mm_H7.0mm_P2.00mm, F.Cu at (111.3, 134.6)
- added C511: 100n, Capacitor_SMD:C_1206_3216Metric_Pad1.42x1.75mm_HandSolder, F.Cu at (122.0, 122.4)
- added C512: 100n, Capacitor_SMD:C_1206_3216Metric_Pad1.42x1.75mm_HandSolder, F.Cu at (122.0, 125.7)
- added C513: 100n, Capacitor_SMD:C_1206_3216Metric_Pad1.42x1.75mm_HandSolder, F.Cu at (128.0, 122.4)
- added C514: 100n, Capacitor_SMD:C_1206_3216Metric_Pad1.42x1.75mm_HandSolder, F.Cu at (128.0, 125.7)
- C105: renamed from C104; value 47p -> 27p
- C106: value 47p -> 27p
- C205: renamed from C11; value 47p -> 27p
- C206: renamed from C12; value 47p -> 27p
- moved R113 32.7 mm to (71.2, 106.2), turned to 270 degrees
- moved R114 29.9 mm to (77.8, 106.2), turned to 270 degrees
- moved Q105 24.9 mm to (62.8, 100.0), turned to 0 degrees
- moved Q106 23.0 mm to (74.5, 106.2), turned to 180 degrees
- moved R110 22.9 mm to (77.0, 118.8), turned to 90 degrees
- moved R112 22.6 mm to (57.0, 100.0), turned to 270 degrees
- moved Q107 20.3 mm to (72.5, 100.0), turned to 180 degrees
- moved Q103 18.7 mm to (74.0, 118.8), turned to 90 degrees
- moved R111 17.3 mm to (74.5, 115.2), turned to 180 degrees
- moved R108 12.0 mm to (71.0, 116.8), turned to 90 degrees
- moved Q101 8.36 mm to (67.5, 113.0)
- moved R109 8.36 mm to (67.5, 120.2), turned to 180 degrees
- moved C105 8.14 mm to (67.5, 109.5), turned to 0 degrees
- moved Q102 7.29 mm to (67.5, 116.8)
- moved R106 6.72 mm to (63.5, 113.5), turned to 180 degrees
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- renumbered C101 to C103, C102 to C104, C7 to C203, C8 to C204, J2 to J201, J4 to J202, R109 to R108, R110 to R109, R111 to R110, R112 to R111, R113 to R112, R114 to R113, R115 to R114, R117 to R115, R118 to R116, R120 to R117, R121 to R118, R122 to R119, R123 to R120, R124 to R121, R125 to R122, R126 to R123, R28 to R201, R29 to R202, R30 to R203, R31 to R204, R32 to R205, R33 to R206
Connections:
- net Net-(C104-Pad2) renamed /ch1/CH1+_FB
- net Net-(C106-Pad2) renamed /ch1/CH1-_FB
- net Net-(C11-Pad2) renamed /ch2/CH2+_FB
- net Net-(C12-Pad2) renamed /ch2/CH2-_FB
- C105 pad 1: Net-(C104-Pad1) -> CH1OUT+
- C106 pad 1: Net-(C106-Pad1) -> CH1OUT-
- C205 pad 1: Net-(C11-Pad1) -> CH2OUT+
- C206 pad 1: Net-(C12-Pad1) -> CH2OUT-
- J101 pad 2: Net-(J101-Pad2) -> Net-(C101-Pad2)
- J101 pad 3: Net-(J101-Pad3) -> Net-(C102-Pad2)
- J201 pad 2: Net-(J2-Pad2) -> Net-(C201-Pad2)
- J201 pad 3: Net-(J2-Pad3) -> Net-(C202-Pad2)
- Q102 pad 4: Net-(C104-Pad1) -> CH1OUT+
- Q105 pad 2: Net-(C104-Pad1) -> CH1OUT+
- Q107 pad 2: Net-(C104-Pad1) -> CH1OUT+
- Q112 pad 4: Net-(C106-Pad1) -> CH1OUT-
- Q115 pad 2: Net-(C106-Pad1) -> CH1OUT-
- Q117 pad 2: Net-(C106-Pad1) -> CH1OUT-
- Q202 pad 4: Net-(C11-Pad1) -> CH2OUT+
- Q205 pad 2: Net-(C11-Pad1) -> CH2OUT+
- Q207 pad 2: Net-(C11-Pad1) -> CH2OUT+
- Q212 pad 4: Net-(C12-Pad1) -> CH2OUT-
- Q215 pad 2: Net-(C12-Pad1) -> CH2OUT-
- Q217 pad 2: Net-(C12-Pad1) -> CH2OUT-
- R101 pad 2: Net-(J101-Pad2) -> Net-(C101-Pad1)
- R102 pad 2: Net-(J101-Pad3) -> Net-(C102-Pad1)
- R201 pad 2: Net-(J2-Pad2) -> Net-(C201-Pad1)
- R202 pad 2: Net-(J2-Pad3) -> Net-(C202-Pad1)
Routing:
- net CH1OUT+: track 0.00 -> 36.8 mm
- net Net-(Q101-Pad2): track 17.0 -> 7.17 mm
- net Net-(Q106-Pad3): track 0.00 -> 7.52 mm
- net /ch1/CH1IN+: track 13.0 -> 5.94 mm
- net Net-(Q103-Pad6): track 12.5 -> 6.76 mm
- net /ch1/CH1+_FB: track 20.9 -> 17.3 mm
- net +15V: track 2.88 -> 0.00 mm
- net -15V: track 2.46 -> 5.19 mm
- net Net-(C103-Pad2): track 2.50 -> 0.00 mm
- net Net-(Q106-Pad1): track 0.00 -> 2.28 mm
- net Net-(Q101-Pad3): track 2.63 -> 4.86 mm
- net Net-(Q101-Pad6): track 2.91 -> 2.09 mm

Commit message: pcb layout
Parts:
- moved C307 185.9 mm to (61.0, 100.0), turned to 180 degrees
- moved C308 177.0 mm to (71.5, 106.8)
- moved C310 161.3 mm to (90.5, 106.8)
- moved D304 160.9 mm to (79.2, 42.5)
- moved C309 158.3 mm to (81.0, 100.0), turned to 180 degrees
- moved C306 150.8 mm to (77.2, 54.0)
- moved R303 145.0 mm to (95.0, 67.5)
- moved R304 143.8 mm to (95.0, 70.5)
- moved C304 143.2 mm to (91.2, 55.0)
- moved D302 127.2 mm to (84.5, 63.2)
- moved U302 126.8 mm to (91.5, 41.8)
- moved C302 124.5 mm to (94.2, 62.2)
- moved R302 122.6 mm to (119.8, 66.0)
- moved D303 115.9 mm to (111.8, 51.0)
- moved R301 115.5 mm to (118.5, 62.2)
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- renumbered C503 to C303, C504 to C304, C505 to C305, C506 to C306, C507 to C307, C508 to C308, C509 to C309, C510 to C310, C511 to C311, C512 to C312, C513 to C313, C514 to C314, R501 to R301, R502 to R302, R503 to R303, R504 to R304
Routing:
- net +15V: track 0.00 -> 79.7 mm, vias 0 -> 4
- net -15V: track 5.19 -> 65.6 mm
- net CH1OUT-: track 0.00 -> 51.3 mm
- net CH1OUT+: track 36.8 -> 55.7 mm
- net /ch1/CH1-_FB: track 0.00 -> 17.8 mm
- net GND: track 0.00 -> 16.6 mm, vias 0 -> 85
- net Net-(C102-Pad2): track 0.00 -> 15.8 mm
- net Net-(C101-Pad2): track 0.00 -> 14.6 mm
- net Net-(Q104-Pad2): track 0.00 -> 14.4 mm
- net /ch1/CH1IN-: track 0.00 -> 10.1 mm
- net Net-(Q111-Pad2): track 0.00 -> 9.75 mm
- net Net-(Q114-Pad2): track 0.00 -> 8.36 mm
- net Net-(Q113-Pad6): track 0.00 -> 8.25 mm
- net Net-(Q116-Pad1): track 0.00 -> 8.17 mm
- net Net-(Q116-Pad3): track 0.00 -> 6.21 mm
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
Commit message: minor changes
Parts:
- moved R36 58.8 mm to (163.8, 115.5)
- moved C203 46.4 mm to (131.5, 122.0)
- moved R41 45.6 mm to (124.2, 102.2)
- moved R37 45.0 mm to (127.2, 104.8)
- moved R203 42.9 mm to (138.2, 122.0)
- moved R205 42.1 mm to (134.8, 122.7)
- moved R202 41.1 mm to (152.8, 120.5)
- moved R34 38.7 mm to (133.8, 117.0)
- moved C206 34.4 mm to (143.5, 96.5)
- moved C204 34.1 mm to (157.0, 118.2)
- moved R50 32.0 mm to (139.0, 98.2)
- moved R47 29.8 mm to (132.5, 93.8)
- moved R44 25.2 mm to (129.8, 109.0)
- moved Q203 23.8 mm to (121.5, 105.5)
- moved Q202 23.5 mm to (128.8, 117.0)
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